Commit message: Adapt Jazzy dual robot cell tutorial for ROS 2 Humble

File: my_dual_robot_cell/my_dual_robot_cell_control/urdf/my_dual_robot_cell_controlled.urdf.xacro (robot description, xacro)
@@ -2,31 +2,33 @@
 <robot name="my_dual_robot_cell" xmlns:xacro="http://ros.org/wiki/xacro">
   <!--First, include the macro from our custom description-->
+  <!-- <xacro:include
+    filename="$(find my_dual_robot_cell_description)/urdf/my_dual_robot_cell_tube_jig_macro.xacro" /> -->
   <xacro:include
-    filename="$(find my_dual_robot_cell_description)/urdf/my_dual_robot_cell_macro.xacro" />
+    filename="$(find my_dual_robot_cell_description)/urdf/my_dual_robot_cell_tube_empty_macro.xacro" />
   <!--The driver already provides a control tag for the UR arm, we can directly include-->
-  <xacro:include filename="$(find ur_robot_driver)/urdf/ur.ros2_control.xacro" />
+  <xacro:include filename="$(find my_dual_robot_cell_description)/urdf/ur.ros2_control.xacro" />
   <!--We need to specify the arguments used for parametrizing our description-->
-  <xacro:arg name="alice_ur_type" default="ur3e" />
-  <xacro:arg name="alice_joint_limits_parameters_file" default="$(find ur_description)/config/$(arg alice_ur_type)/joint_limits.yaml" />
-  <xacro:arg name="alice_kinematics_parameters_file" default="$(find ur_description)/config/$(arg alice_ur_type)/default_kinematics.yaml" />
-  <xacro:arg name="alice_physical_parameters_file" default="$(find ur_description)/config/$(arg alice_ur_type)/physical_parameters.yaml" />
-  <xacro:arg name="alice_visual_parameters_file" default="$(find ur_description)/config/$(arg alice_ur_type)/visual_parameters.yaml" />
+  <xacro:arg name="alice_ur_type" default="ur5e" />
+  <xacro:arg name="alice_joint_limits_parameters_file" default="$(find my_dual_robot_cell_description)/config/$(arg alice_ur_type)/joint_limits.yaml" />
+  <xacro:arg name="alice_kinematics_parameters_file" default="$(find my_dual_robot_cell_description)/config/$(arg alice_ur_type)/default_kinematics.yaml" />
+  <xacro:arg name="alice_physical_parameters_file" default="$(find my_dual_robot_cell_description)/config/$(arg alice_ur_type)/physical_parameters.yaml" />
+  <xacro:arg name="alice_visual_parameters_file" default="$(find my_dual_robot_cell_description)/config/$(arg alice_ur_type)/visual_parameters.yaml" />
   <xacro:arg name="bob_ur_type" default="ur5e" />
-  <xacro:arg name="bob_joint_limits_parameters_file" default="$(find ur_description)/config/$(arg bob_ur_type)/joint_limits.yaml" />
-  <xacro:arg name="bob_kinematics_parameters_file" default="$(find ur_description)/config/$(arg bob_ur_type)/default_kinematics.yaml" />
-  <xacro:arg name="bob_physical_parameters_file" default="$(find ur_description)/config/$(arg bob_ur_type)/physical_parameters.yaml" />
-  <xacro:arg name="bob_visual_parameters_file" default="$(find ur_description)/config/$(arg bob_ur_type)/visual_parameters.yaml" />
+  <xacro:arg name="bob_joint_limits_parameters_file" default="$(find my_dual_robot_cell_description)/config/$(arg bob_ur_type)/joint_limits.yaml" />
+  <xacro:arg name="bob_kinematics_parameters_file" default="$(find my_dual_robot_cell_description)/config/$(arg bob_ur_type)/default_kinematics.yaml" />
+  <xacro:arg name="bob_physical_parameters_file" default="$(find my_dual_robot_cell_description)/config/$(arg bob_ur_type)/physical_parameters.yaml" />
+  <xacro:arg name="bob_visual_parameters_file" default="$(find my_dual_robot_cell_description)/config/$(arg bob_ur_type)/visual_parameters.yaml" />
   <xacro:arg name="alice_use_mock_hardware" default="false" />
   <xacro:arg name="alice_mock_sensor_commands" default="false" />
-  <xacro:arg name="alice_robot_ip" default="192.168.57.101" />
+  <xacro:arg name="alice_robot_ip" default="192.168.1.4" />
   <xacro:arg name="alice_reverse_port" default="50006" />
   <xacro:arg name="alice_script_sender_port" default="50007" />
-  <xacro:arg name="alice_script_command_port" default="50010" />
+  <xacro:arg name="alice_script_command_port" default="50002" />
   <xacro:arg name="alice_trajectory_port" default="50009" />
   <xacro:arg name="bob_use_mock_hardware" default="false" />
   <xacro:arg name="bob_mock_sensor_commands" default="false" />
-  <xacro:arg name="bob_robot_ip" default="192.168.57.100" />
-  <xacro:arg name="bob_reverse_port" default="50001" />
-  <xacro:arg name="bob_script_sender_port" default="50002" />
+  <xacro:arg name="bob_robot_ip" default="192.168.1.6" />
+  <xacro:arg name="bob_reverse_port" default="50005" />
+  <xacro:arg name="bob_script_sender_port" default="50008" />
   <xacro:arg name="bob_script_command_port" default="50004" />
   <xacro:arg name="bob_trajectory_port" default="50003" />
@@ -35,4 +37,8 @@
   <xacro:arg name="ur_output_recipe_filename" default="$(find ur_robot_driver)/resources/rtde_output_recipe.txt" />
   <xacro:arg name="ur_input_recipe_filename" default="$(find ur_robot_driver)/resources/rtde_input_recipe.txt" />
+  <xacro:property name="alice_kinematics_params_file" value="$(arg alice_kinematics_parameters_file)"/>
+  <xacro:property name="alice_kinematics_hash" value="${xacro.load_yaml(alice_kinematics_params_file)['kinematics']['hash']}"/>
+  <xacro:property name="bob_kinematics_params_file" value="$(arg bob_kinematics_parameters_file)"/>
+  <xacro:property name="bob_kinematics_hash" value="${xacro.load_yaml(bob_kinematics_params_file)['kinematics']['hash']}"/>
   <link name="world" />
   <xacro:my_dual_robot_cell
@@ -48,4 +54,12 @@
     bob_physical_parameters_file="$(arg bob_physical_parameters_file)"
     bob_visual_parameters_file="$(arg bob_visual_parameters_file)"
+    bob_reverse_port="$(arg bob_reverse_port)"
+    alice_reverse_port="$(arg alice_reverse_port)"
+    alice_trajectory_port="$(arg alice_trajectory_port)"
+    alice_script_sender_port="$(arg alice_script_sender_port)"
+    alice_script_command_port="$(arg alice_script_command_port)"
+    bob_trajectory_port="$(arg bob_trajectory_port)"
+    bob_script_sender_port="$(arg bob_script_sender_port)"
+    bob_script_command_port="$(arg bob_script_command_port)"
   >
     <origin xyz="0 0 1" rpy="0 0 0" />
@@ -54,32 +68,32 @@
     name="alice"
     tf_prefix="alice_"
-    kinematics_parameters_file="$(arg alice_kinematics_parameters_file)"
+    hash_kinematics="${alice_kinematics_hash}"
     robot_ip="$(arg alice_robot_ip)"
     script_filename="$(arg ur_script_filename)"
     output_recipe_filename="$(arg ur_output_recipe_filename)"
     input_recipe_filename="$(arg ur_input_recipe_filename)"
-    use_mock_hardware="$(arg alice_use_mock_hardware)"
-    mock_sensor_commands="$(arg alice_mock_sensor_commands)"
+    use_fake_hardware="$(arg alice_use_mock_hardware)"
+    fake_sensor_commands="$(arg alice_mock_sensor_commands)"
     headless_mode="$(arg headless_mode)"
     reverse_port="$(arg alice_reverse_port)"
+    trajectory_port="$(arg alice_trajectory_port)"
     script_sender_port="$(arg alice_script_sender_port)"
     script_command_port="$(arg alice_script_command_port)"
-    trajectory_port="$(arg alice_trajectory_port)"
   />
   <xacro:ur_ros2_control
     name="bob"
     tf_prefix="bob_"
-    kinematics_parameters_file="$(arg bob_kinematics_parameters_file)"
+    hash_kinematics="${bob_kinematics_hash}"
     robot_ip="$(arg bob_robot_ip)"
     script_filename="$(arg ur_script_filename)"
     output_recipe_filename="$(arg ur_output_recipe_filename)"
     input_recipe_filename="$(arg ur_input_recipe_filename)"
-    use_mock_hardware="$(arg bob_use_mock_hardware)"
-    mock_sensor_commands="$(arg bob_mock_sensor_commands)"
+    use_fake_hardware="$(arg bob_use_mock_hardware)"
+    fake_sensor_commands="$(arg bob_mock_sensor_commands)"
     headless_mode="$(arg headless_mode)"
     reverse_port="$(arg bob_reverse_port)"
+    trajectory_port="$(arg bob_trajectory_port)"
     script_sender_port="$(arg bob_script_sender_port)"
     script_command_port="$(arg bob_script_command_port)"
-    trajectory_port="$(arg bob_trajectory_port)"
   />
 </robot>

File: my_dual_robot_cell/my_dual_robot_cell_description/urdf/my_dual_robot_cell.urdf.xacro (robot description, xacro)
@@ -2,14 +2,23 @@
 <robot name="my_dual_robot_cell" xmlns:xacro="http://ros.org/wiki/xacro">
   <xacro:include filename="$(find my_dual_robot_cell_description)/urdf/my_dual_robot_cell_macro.xacro"/>
-  <xacro:arg name="alice_ur_type" default="ur3e"/>
-  <xacro:arg name="alice_joint_limits_parameters_file" default="$(find ur_description)/config/$(arg alice_ur_type)/joint_limits.yaml"/>
-  <xacro:arg name="alice_kinematics_parameters_file" default="$(find ur_description)/config/$(arg alice_ur_type)/default_kinematics.yaml"/>
-  <xacro:arg name="alice_physical_parameters_file" default="$(find ur_description)/config/$(arg alice_ur_type)/physical_parameters.yaml"/>
-  <xacro:arg name="alice_visual_parameters_file" default="$(find ur_description)/config/$(arg alice_ur_type)/visual_parameters.yaml"/>
+  <xacro:arg name="alice_ur_type" default="ur5e"/>
+  <xacro:arg name="alice_joint_limits_parameters_file" default="$(find my_dual_robot_cell_description)/config/$(arg alice_ur_type)/joint_limits.yaml"/>
+  <xacro:arg name="alice_kinematics_parameters_file" default="$(find my_dual_robot_cell_description)/config/$(arg alice_ur_type)/default_kinematics.yaml"/>
+  <xacro:arg name="alice_physical_parameters_file" default="$(find my_dual_robot_cell_description)/config/$(arg alice_ur_type)/physical_parameters.yaml"/>
+  <xacro:arg name="alice_visual_parameters_file" default="$(find my_dual_robot_cell_description)/config/$(arg alice_ur_type)/visual_parameters.yaml"/>
   <xacro:arg name="bob_ur_type" default="ur5e"/>
-  <xacro:arg name="bob_joint_limits_parameters_file" default="$(find ur_description)/config/$(arg bob_ur_type)/joint_limits.yaml"/>
-  <xacro:arg name="bob_kinematics_parameters_file" default="$(find ur_description)/config/$(arg bob_ur_type)/default_kinematics.yaml"/>
-  <xacro:arg name="bob_physical_parameters_file" default="$(find ur_description)/config/$(arg bob_ur_type)/physical_parameters.yaml"/>
-  <xacro:arg name="bob_visual_parameters_file" default="$(find ur_description)/config/$(arg bob_ur_type)/visual_parameters.yaml"/>
+  <xacro:arg name="bob_joint_limits_parameters_file" default="$(find my_dual_robot_cell_description)/config/$(arg bob_ur_type)/joint_limits.yaml"/>
+  <xacro:arg name="bob_kinematics_parameters_file" default="$(find my_dual_robot_cell_description)/config/$(arg bob_ur_type)/default_kinematics.yaml"/>
+  <xacro:arg name="bob_physical_parameters_file" default="$(find my_dual_robot_cell_description)/config/$(arg bob_ur_type)/physical_parameters.yaml"/>
+  <xacro:arg name="bob_visual_parameters_file" default="$(find my_dual_robot_cell_description)/config/$(arg bob_ur_type)/visual_parameters.yaml"/>
+  <xacro:include filename="$(find my_dual_robot_cell_description)/urdf/ur_macro.xacro"/>
+  <xacro:arg name="alice_reverse_port" default="50006"/>
+  <xacro:arg name="alice_trajectory_port" default="50009"/>
+  <xacro:arg name="alice_script_command_port" default="50002"/>
+  <xacro:arg name="alice_script_sender_port" default="50007"/>
+  <xacro:arg name="bob_reverse_port" default="50005"/>
+  <xacro:arg name="bob_trajectory_port" default="50003"/>
+  <xacro:arg name="bob_script_command_port" default="50004"/>
+  <xacro:arg name="bob_script_sender_port" default="50008"/>
   <link name="world"/>
   <!--This will create the scene where the robots are located in-->
@@ -21,4 +30,12 @@
     alice_physical_parameters_file="$(arg alice_physical_parameters_file)"
     alice_visual_parameters_file="$(arg alice_visual_parameters_file)"
+    alice_reverse_port="$(arg alice_reverse_port)"
+    bob_reverse_port="$(arg bob_reverse_port)"
+    alice_trajectory_port="$(arg alice_trajectory_port)"
+    bob_trajectory_port="$(arg bob_trajectory_port)"
+    alice_script_command_port="$(arg alice_script_command_port)"
+    bob_script_command_port="$(arg bob_script_command_port)"
+    alice_script_sender_port="$(arg alice_script_sender_port)"
+    bob_script_sender_port="$(arg bob_script_sender_port)"
     bob_ur_type="$(arg bob_ur_type)"
     bob_joint_limits_parameters_file="$(arg bob_joint_limits_parameters_file)"
@@ -27,5 +44,5 @@
     bob_visual_parameters_file="$(arg bob_visual_parameters_file)"
     >
-      <origin xyz="0 0 1" rpy="0 0 0" />
+      <origin xyz="0 0 0" rpy="0 0 0" />
   </xacro:my_dual_robot_cell>
 </robot>

File: my_dual_robot_cell/my_dual_robot_cell_description/urdf/my_dual_robot_cell_macro.xacro (robot description, xacro)
@@ -1,5 +1,13 @@
 <?xml version="1.0"?>
 <robot xmlns:xacro="http://ros.org/wiki/xacro">
-  <xacro:include filename="$(find ur_description)/urdf/ur_macro.xacro"/>
+  <xacro:include filename="$(find my_dual_robot_cell_description)/urdf/ur_macro.xacro"/>
+  <xacro:arg name="alice_reverse_port" default="50006"/>
+  <xacro:arg name="alice_trajectory_port" default="50009"/>
+  <xacro:arg name="alice_script_command_port" default="50002"/>
+  <xacro:arg name="alice_script_sender_port" default="50007"/>
+  <xacro:arg name="bob_reverse_port" default="50005"/>
+  <xacro:arg name="bob_trajectory_port" default="50003"/>
+  <xacro:arg name="bob_script_command_port" default="50004"/>
+  <xacro:arg name="bob_script_sender_port" default="50008"/>
   <xacro:macro name="my_dual_robot_cell" params="
     parent
@@ -10,4 +18,8 @@
     alice_physical_parameters_file
     alice_visual_parameters_file
+    alice_reverse_port
+    alice_trajectory_port
+    alice_script_command_port
+    alice_script_sender_port
     bob_ur_type
     bob_joint_limits_parameters_file
@@ -15,4 +27,8 @@
     bob_physical_parameters_file
     bob_visual_parameters_file
+    bob_reverse_port
+    bob_trajectory_port
+    bob_script_command_port
+    bob_script_sender_port
     ">
     <joint name="table_base_joint" type="fixed">
@@ -20,62 +36,38 @@
       <parent link="${parent}" />
       <child link="table" />
+      <origin xyz="0.0 0.0 0" rpy="0 0 0" />
     </joint>
     <link name="table">
       <visual>
         <geometry>
-          <mesh filename="package://my_robot_cell_description/meshes/fzi_table.dae"/>
+          <mesh filename="package://my_robot_cell_description/meshes/frame_wo_screw_basetrans_m.dae"/>
         </geometry>
-        <origin rpy="0 0 0" xyz="0.75 0.5 -1"/>
+        <origin rpy="0 0 0" xyz="0.0 0.0 0"/>
       </visual>
       <collision>
         <geometry>
-          <mesh filename="package://my_robot_cell_description/meshes/fzi_table.dae"/>
+          <mesh filename="package://my_robot_cell_description/meshes/frame_wo_screw_basetrans_m.stl"/>
         </geometry>
-        <origin rpy="0 0 0" xyz="0.75 0.5 -1"/>
+        <origin rpy="0 0 0" xyz="0.0 0.0 0"/>
       </collision>
     </link>
-    <link name="monitor">
-      <visual>
-        <geometry>
-          <mesh filename="package://my_robot_cell_description/meshes/171005_Motek_Monitor_L.dae"/>
-        </geometry>
-      </visual>
-      <collision>
-        <geometry>
-          <mesh filename="package://my_robot_cell_description/meshes/171005_Motek_Monitor_L.dae"/>
-        </geometry>
-      </collision>
-    </link>
-    <joint name="base_to_monitor" type="fixed">
-      <parent link="table"/>
-      <child link="monitor"/>
-      <origin xyz="0.2 0.6 0"/>
-    </joint>
-    <material name="white">
-      <color rgba="1 1 1 1"/>
-    </material>
-    <link name="wall">
-      <visual>
-        <geometry>
-          <mesh filename="package://my_robot_cell_description/meshes/wall.dae"/>
-        </geometry>
-      </visual>
-      <collision>
-        <geometry>
-          <box size="4.44 0.1 2.5"/>
-        </geometry>
-      </collision>
-    </link>
-    <joint name="base_to_wall" type="fixed">
-      <parent link="table"/>
-      <child link="wall"/>
-      <origin xyz="1.25 1.5 0.5"/>
-    </joint>
     <!--Creates the mounts to attach the robots to the table-->
     <link name="alice_robot_mount"/>
+    <joint name="base_to_alice_robot_mount" type="floating">
+      <parent link="table"/>
+      <child link="alice_robot_mount"/>
+      <origin xyz="-0.25 0.0 0" rpy="0 0 0" />
+    </joint>
+    <link name="bob_robot_mount"/>
+    <joint name="base_to_bob_robot_mount" type="floating">
+      <parent link="table"/>
+      <child link="bob_robot_mount"/>
+      <origin xyz="0.25 0.0 0" rpy="0 0 0" />
+    </joint>
+    <!-- <link name="alice_robot_mount"/>
     <joint name="base_to_alice_robot_mount" type="fixed">
       <parent link="table"/>
       <child link="alice_robot_mount"/>
-      <origin xyz="0.2 0.3 0" rpy="0 0 ${pi}" />
+      <origin xyz="-0.25 0.0 0" rpy="0 0 0" />
     </joint>
     <link name="bob_robot_mount"/>
@@ -83,6 +75,6 @@
       <parent link="table"/>
       <child link="bob_robot_mount"/>
-      <origin xyz="1.2 0.3 0" rpy="0 0 ${pi}" />
-    </joint>
+      <origin xyz="0.25 0.0 0" rpy="0 0 0" />
+    </joint> -->
     <!--Creates the 1st Robot-->
     <xacro:ur_robot
@@ -94,4 +86,9 @@
       physical_parameters_file="${alice_physical_parameters_file}"
       visual_parameters_file="${alice_visual_parameters_file}"
+      generate_ros2_control_tag="false"
+      reverse_port="${alice_reverse_port}"
+      trajectory_port="${alice_trajectory_port}"
+      script_sender_port="${alice_script_sender_port}"
+      script_command_port="${alice_script_command_port}"
     >
       <origin xyz="0 0 0" rpy="0 0 0" />
@@ -106,4 +103,9 @@
       physical_parameters_file="${bob_physical_parameters_file}"
       visual_parameters_file="${bob_visual_parameters_file}"
+      generate_ros2_control_tag="false"
+      reverse_port="${bob_reverse_port}"
+      trajectory_port="${bob_trajectory_port}"
+      script_sender_port="${bob_script_sender_port}"
+      script_command_port="${bob_script_command_port}"
     >
       <origin xyz="0 0 0" rpy="0 0 0" />
